Commit message: Create new folders for humanoid_description xacro files

File: src/robot_description/humanoid_description/urdf/humanoid.urdf.xacro (robot description, xacro)
@@ -6,4 +6,6 @@
   <xacro:include filename="$(find humanoid_description)/xacro/common/inertials.xacro"/>
   <xacro:include filename="$(find humanoid_description)/xacro/common/transmission.xacro"/>
+  <xacro:include filename="$(find humanoid_description)/xacro/joints/robot_joints.xacro"/>
+  <xacro:include filename="$(find humanoid_description)/xacro/links/robot_linksxacro"/>
   <!-- Robot components -->
   <!-- TODO: Uncomment as xacro files are created
@@ -31,9 +33,9 @@
   <!-- ==================== BASE LINK ==================== -->
   <!-- Base footprint (on ground) -->
-  <link name="base_footprint">
+  <!-- <link name="base_footprint">
     <xacro:point_mass m="0.001"/>
-  </link>
+  </link> -->
   <!-- Base link (torso base) -->
-  <link name="base_link">
+  <!-- <link name="base_link">
     <visual>
       <origin xyz="0 0 0" rpy="0 0 0"/>
@@ -48,14 +50,14 @@
         <box size="${torso_depth} ${torso_width} ${torso_height}"/>
       </geometry>
-    </collision>
+    </collision> -->
     <!-- TODO: Replace with actual inertial values -->
-    <xacro:box_inertia m="10.0" x="${torso_depth}" y="${torso_width}" z="${torso_height}"/>
-  </link>
+    <!-- <xacro:box_inertia m="10.0" x="${torso_depth}" y="${torso_width}" z="${torso_height}"/>
+  </link> -->
   <!-- Base footprint to base link joint -->
-  <joint name="base_footprint_joint" type="fixed">
+  <!-- <joint name="base_footprint_joint" type="fixed">
     <parent link="base_footprint"/>
     <child link="base_link"/>
     <origin xyz="0 0 0.5" rpy="0 0 0"/>
-  </joint>
+  </joint> -->
   <!-- ==================== COMPONENT INSTANTIATION ==================== -->
   <!-- TODO: Instantiate robot components here -->

Commit message: Add base_link to robot

File: src/robot_description/humanoid_description/urdf/humanoid.urdf.xacro (robot description, xacro)
@@ -32,32 +32,33 @@
   <xacro:property name="joint_velocity_limit" value="2.0"/>
   <!-- ==================== BASE LINK ==================== -->
-  <!-- Base footprint (on ground) -->
-  <!-- <link name="base_footprint">
-    <xacro:point_mass m="0.001"/>
-  </link> -->
-  <!-- Base link (torso base) -->
-  <!-- <link name="base_link">
+ <link name="base_link">
+    <inertial>
+      <origin xyz="0 0 0" rpy="0 0 0"/>
+      <mass value="0.001"/>
+      <inertia ixx="0.000001" ixy="0" ixz="0" iyy="0.000001" iyz="0" izz="0.000002"/>
+    </inertial>
     <visual>
       <origin xyz="0 0 0" rpy="0 0 0"/>
       <geometry>
-        <box size="${torso_depth} ${torso_width} ${torso_height}"/>
+        <sphere radius="0.01"/>
       </geometry>
-      <material name="robot_body"/>
+      <material name="">
+        <color rgba="1 0 0 1"/>
+      </material>
     </visual>
     <collision>
       <origin xyz="0 0 0" rpy="0 0 0"/>
       <geometry>
-        <box size="${torso_depth} ${torso_width} ${torso_height}"/>
+        <sphere radius="0.01"/>
       </geometry>
-    </collision> -->
-    <!-- TODO: Replace with actual inertial values -->
-    <!-- <xacro:box_inertia m="10.0" x="${torso_depth}" y="${torso_width}" z="${torso_height}"/>
-  </link> -->
-  <!-- Base footprint to base link joint -->
-  <!-- <joint name="base_footprint_joint" type="fixed">
-    <parent link="base_footprint"/>
-    <child link="base_link"/>
-    <origin xyz="0 0 0.5" rpy="0 0 0"/>
-  </joint> -->
+    </collision>
+  </link>
+  <!-- Fixed joint from base_link to base (leg structure root) -->
+  <!-- This joint lifts the leg structure so feet are at ground level (z=0) -->
+  <joint name="base_link_to_base" type="fixed">
+    <parent link="base_link"/>
+    <child link="base"/>
+    <origin xyz="0 0 0.813" rpy="0 0 0"/>
+  </joint>
   <!-- ==================== COMPONENT INSTANTIATION ==================== -->
   <!-- TODO: Instantiate robot components here -->

Commit message: Feat: Add controller launch inclusion to gazebo launch file

File: src/robot_description/humanoid_description/urdf/humanoid.urdf.xacro (robot description, xacro)
@@ -33,9 +33,4 @@
   <!-- ==================== BASE LINK ==================== -->
  <link name="base_link">
-    <inertial>
-      <origin xyz="0 0 0" rpy="0 0 0"/>
-      <mass value="0.001"/>
-      <inertia ixx="0.000001" ixy="0" ixz="0" iyy="0.000001" iyz="0" izz="0.000002"/>
-    </inertial>
     <visual>
       <origin xyz="0 0 0" rpy="0 0 0"/>
@@ -47,10 +42,4 @@
       </material>
     </visual>
-    <collision>
-      <origin xyz="0 0 0" rpy="0 0 0"/>
-      <geometry>
-        <sphere radius="0.01"/>
-      </geometry>
-    </collision>
   </link>
   <!-- Fixed joint from base_link to base (leg structure root) -->
@@ -95,11 +84,116 @@
   <!-- <xacro:imu parent="torso_link"/> -->
   <!-- ==================== ROS2_CONTROL ==================== -->
-  <!-- TODO: Add ros2_control hardware interface configuration -->
-  <!--
-  <ros2_control name="humanoid_hardware" type="system">
+  <ros2_control name="GazeboSystem" type="system">
     <hardware>
-      <plugin>humanoid_hardware/HumanoidHardwareInterface</plugin>
+      <plugin>gz_ros2_control/GazeboSimSystem</plugin>
     </hardware>
+    <!-- Leg joints -->
+    <joint name="dof_left_hip_pitch_04">
+      <command_interface name="position"/>
+      <state_interface name="position"/>
+      <state_interface name="velocity"/>
+    </joint>
+    <joint name="dof_left_hip_roll_03">
+      <command_interface name="position"/>
+      <state_interface name="position"/>
+      <state_interface name="velocity"/>
+    </joint>
+    <joint name="dof_left_hip_yaw_03">
+      <command_interface name="position"/>
+      <state_interface name="position"/>
+      <state_interface name="velocity"/>
+    </joint>
+    <joint name="dof_left_knee_04">
+      <command_interface name="position"/>
+      <state_interface name="position"/>
+      <state_interface name="velocity"/>
+    </joint>
+    <joint name="dof_left_ankle_02">
+      <command_interface name="position"/>
+      <state_interface name="position"/>
+      <state_interface name="velocity"/>
+    </joint>
+    <joint name="dof_right_hip_pitch_04">
+      <command_interface name="position"/>
+      <state_interface name="position"/>
+      <state_interface name="velocity"/>
+    </joint>
+    <joint name="dof_right_hip_roll_03">
+      <command_interface name="position"/>
+      <state_interface name="position"/>
+      <state_interface name="velocity"/>
+    </joint>
+    <joint name="dof_right_hip_yaw_03">
+      <command_interface name="position"/>
+      <state_interface name="position"/>
+      <state_interface name="velocity"/>
+    </joint>
+    <joint name="dof_right_knee_04">
+      <command_interface name="position"/>
+      <state_interface name="position"/>
+      <state_interface name="velocity"/>
+    </joint>
+    <joint name="dof_right_ankle_02">
+      <command_interface name="position"/>
+      <state_interface name="position"/>
+      <state_interface name="velocity"/>
+    </joint>
+    <!-- Arm joints -->
+    <joint name="dof_left_shoulder_pitch_03">
+      <command_interface name="position"/>
+      <state_interface name="position"/>
+      <state_interface name="velocity"/>
+    </joint>
+    <joint name="dof_left_shoulder_roll_03">
+      <command_interface name="position"/>
+      <state_interface name="position"/>
+      <state_interface name="velocity"/>
+    </joint>
+    <joint name="dof_left_shoulder_yaw_02">
+      <command_interface name="position"/>
+      <state_interface name="position"/>
+      <state_interface name="velocity"/>
+    </joint>
+    <joint name="dof_left_elbow_02">
+      <command_interface name="position"/>
+      <state_interface name="position"/>
+      <state_interface name="velocity"/>
+    </joint>
+    <joint name="dof_left_wrist_00">
+      <command_interface name="position"/>
+      <state_interface name="position"/>
+      <state_interface name="velocity"/>
+    </joint>
+    <joint name="dof_right_shoulder_pitch_03">
+      <command_interface name="position"/>
+      <state_interface name="position"/>
+      <state_interface name="velocity"/>
+    </joint>
+    <joint name="dof_right_shoulder_roll_03">
+      <command_interface name="position"/>
+      <state_interface name="position"/>
+      <state_interface name="velocity"/>
+    </joint>
+    <joint name="dof_right_shoulder_yaw_02">
+      <command_interface name="position"/>
+      <state_interface name="position"/>
+      <state_interface name="velocity"/>
+    </joint>
+    <joint name="dof_right_elbow_02">
+      <command_interface name="position"/>
+      <state_interface name="position"/>
+      <state_interface name="velocity"/>
+    </joint>
+    <joint name="dof_right_wrist_00">
+      <command_interface name="position"/>
+      <state_interface name="position"/>
+      <state_interface name="velocity"/>
+    </joint>
   </ros2_control>
-  -->
+  <!-- Gazebo ros2_control plugin -->
+  <gazebo>
+    <plugin filename="gz_ros2_control-system" name="gz_ros2_control::GazeboSimROS2ControlPlugin">
+      <parameters>$(find humanoid_gazebo)/config/controllers.yaml</parameters>
+    </plugin>
+  </gazebo>
 </robot>

Commit message: refactor urdf for ros2 control  and gazebo plugin

File: src/robot_description/humanoid_description/urdf/humanoid.urdf.xacro (robot description, xacro)
@@ -6,4 +6,6 @@
   <xacro:include filename="$(find humanoid_description)/xacro/common/inertials.xacro"/>
   <xacro:include filename="$(find humanoid_description)/xacro/common/transmission.xacro"/>
+  <xacro:include filename="$(find humanoid_description)/xacro/common/ros2_control.xacro"/>
+  <xacro:include filename="$(find humanoid_description)/xacro/common/gazebo.xacro"/>
   <xacro:include filename="$(find humanoid_description)/xacro/joints/robot_joints.xacro"/>
   <xacro:include filename="$(find humanoid_description)/xacro/links/robot_links.xacro"/>
@@ -83,117 +85,3 @@
   <!-- <xacro:cameras parent="head_link"/> -->
   <!-- <xacro:imu parent="torso_link"/> -->
-  <!-- ==================== ROS2_CONTROL ==================== -->
-  <ros2_control name="GazeboSystem" type="system">
-    <hardware>
-      <plugin>gz_ros2_control/GazeboSimSystem</plugin>
-    </hardware>
-    <!-- Leg joints -->
-    <joint name="dof_left_hip_pitch_04">
-      <command_interface name="position"/>
-      <state_interface name="position"/>
-      <state_interface name="velocity"/>
-    </joint>
-    <joint name="dof_left_hip_roll_03">
-      <command_interface name="position"/>
-      <state_interface name="position"/>
-      <state_interface name="velocity"/>
-    </joint>
-    <joint name="dof_left_hip_yaw_03">
-      <command_interface name="position"/>
-      <state_interface name="position"/>
-      <state_interface name="velocity"/>
-    </joint>
-    <joint name="dof_left_knee_04">
-      <command_interface name="position"/>
-      <state_interface name="position"/>
-      <state_interface name="velocity"/>
-    </joint>
-    <joint name="dof_left_ankle_02">
-      <command_interface name="position"/>
-      <state_interface name="position"/>
-      <state_interface name="velocity"/>
-    </joint>
-    <joint name="dof_right_hip_pitch_04">
-      <command_interface name="position"/>
-      <state_interface name="position"/>
-      <state_interface name="velocity"/>
-    </joint>
-    <joint name="dof_right_hip_roll_03">
-      <command_interface name="position"/>
-      <state_interface name="position"/>
-      <state_interface name="velocity"/>
-    </joint>
-    <joint name="dof_right_hip_yaw_03">
-      <command_interface name="position"/>
-      <state_interface name="position"/>
-      <state_interface name="velocity"/>
-    </joint>
-    <joint name="dof_right_knee_04">
-      <command_interface name="position"/>
-      <state_interface name="position"/>
-      <state_interface name="velocity"/>
-    </joint>
-    <joint name="dof_right_ankle_02">
-      <command_interface name="position"/>
-      <state_interface name="position"/>
-      <state_interface name="velocity"/>
-    </joint>
-    <!-- Arm joints -->
-    <joint name="dof_left_shoulder_pitch_03">
-      <command_interface name="position"/>
-      <state_interface name="position"/>
-      <state_interface name="velocity"/>
-    </joint>
-    <joint name="dof_left_shoulder_roll_03">
-      <command_interface name="position"/>
-      <state_interface name="position"/>
-      <state_interface name="velocity"/>
-    </joint>
-    <joint name="dof_left_shoulder_yaw_02">
-      <command_interface name="position"/>
-      <state_interface name="position"/>
-      <state_interface name="velocity"/>
-    </joint>
-    <joint name="dof_left_elbow_02">
-      <command_interface name="position"/>
-      <state_interface name="position"/>
-      <state_interface name="velocity"/>
-    </joint>
-    <joint name="dof_left_wrist_00">
-      <command_interface name="position"/>
-      <state_interface name="position"/>
-      <state_interface name="velocity"/>
-    </joint>
-    <joint name="dof_right_shoulder_pitch_03">
-      <command_interface name="position"/>
-      <state_interface name="position"/>
-      <state_interface name="velocity"/>
-    </joint>
-    <joint name="dof_right_shoulder_roll_03">
-      <command_interface name="position"/>
-      <state_interface name="position"/>
-      <state_interface name="velocity"/>
-    </joint>
-    <joint name="dof_right_shoulder_yaw_02">
-      <command_interface name="position"/>
-      <state_interface name="position"/>
-      <state_interface name="velocity"/>
-    </joint>
-    <joint name="dof_right_elbow_02">
-      <command_interface name="position"/>
-      <state_interface name="position"/>
-      <state_interface name="velocity"/>
-    </joint>
-    <joint name="dof_right_wrist_00">
-      <command_interface name="position"/>
-      <state_interface name="position"/>
-      <state_interface name="velocity"/>
-    </joint>
-  </ros2_control>
-  <!-- Gazebo ros2_control plugin -->
-  <gazebo>
-    <plugin filename="gz_ros2_control-system" name="gz_ros2_control::GazeboSimROS2ControlPlugin">
-      <parameters>$(find humanoid_gazebo)/config/controllers.yaml</parameters>
-    </plugin>
-  </gazebo>
 </robot>

Commit message: add 8 force sensors

File: src/robot_description/humanoid_description/urdf/humanoid.urdf.xacro (robot description, xacro)
@@ -36,5 +36,5 @@
   <xacro:property name="joint_velocity_limit" value="2.0"/>
   <!-- ==================== BASE LINK ==================== -->
- <link name="base_link">
+ <!-- <link name="base_link">
     <visual>
       <origin xyz="0 0 0" rpy="0 0 0"/>
@@ -46,12 +46,12 @@
       </material>
     </visual>
-  </link>
+  </link> -->
   <!-- Fixed joint from base_link to base (leg structure root) -->
   <!-- This joint lifts the leg structure so feet are at ground level (z=0) -->
-  <joint name="base_link_to_base" type="fixed">
+  <!-- <joint name="base_link_to_base" type="fixed">
     <parent link="base_link"/>
     <child link="base"/>
     <origin xyz="0 0 0.813" rpy="0 0 0"/>
-  </joint>
+  </joint> -->
   <!-- ==================== COMPONENT INSTANTIATION ==================== -->
   <!-- TODO: Instantiate robot components here -->
@@ -92,12 +92,42 @@
   <xacro:foot_contact_sensor
     foot_link="LFootBushing_GPF_1517_12"
-    prefix="left"
-    foot_bottom_offset="0.1"
+    prefix="left_heel_medial"
+    position="0.061 0.06 0.0055"
+    sensor_rpy="1.5708 0 0"/>
+  <xacro:foot_contact_sensor
+    foot_link="LFootBushing_GPF_1517_12"
+    prefix="left_heel_lateral"
+    position="0.061 0.06 -0.035"
+    sensor_rpy="1.5708 0 0"/>
+  <xacro:foot_contact_sensor
+    foot_link="LFootBushing_GPF_1517_12"
+    prefix="left_toe_medial"
+    position="-0.112 0.06 0.0055"
+    sensor_rpy="1.5708 0 0"/>
+  <xacro:foot_contact_sensor
+    foot_link="LFootBushing_GPF_1517_12"
+    prefix="left_toe_lateral"
+    position="-0.105 0.06 -0.035"
     sensor_rpy="1.5708 0 0"/>
   <!-- Right foot: Z- points down, so rotate -90deg around X to make sensor flat -->
   <xacro:foot_contact_sensor
     foot_link="RFootBushing_GPF_1517_12"
-    prefix="right"
-    foot_bottom_offset="-0.1"
-    sensor_rpy="-1.5708 0 0"/>
+    prefix="right_heel_medial"
+    position="0.061 -0.06 0.0055"
+    sensor_rpy="1.5708 0 0"/>
+  <xacro:foot_contact_sensor
+    foot_link="RFootBushing_GPF_1517_12"
+    prefix="right_heel_lateral"
+    position="0.061 -0.06 -0.035"
+    sensor_rpy="1.5708 0 0"/>
+  <xacro:foot_contact_sensor
+    foot_link="RFootBushing_GPF_1517_12"
+    prefix="right_toe_medial"
+    position="-0.112 -0.06 0.0055"
+    sensor_rpy="1.5708 0 0"/>
+  <xacro:foot_contact_sensor
+    foot_link="RFootBushing_GPF_1517_12"
+    prefix="right_toe_lateral"
+    position="-0.105 -0.06 -0.035"
+    sensor_rpy="1.5708 0 0"/>
 </robot>

File: src/robot_description/humanoid_description/xacro/sensors/force_torque.xacro (robot description, xacro)
@@ -20,5 +20,5 @@
     - update_rate: Sensor update frequency (Hz)
   -->
-  <xacro:macro name="force_torque_sensor" params="parent_link sensor_name topic position:='0 0 0' rpy:='0 0 0' box_size:='0.08 0.06 0.01' update_rate:=100.0">
+  <xacro:macro name="force_torque_sensor" params="parent_link sensor_name topic position:='0 0 0' rpy:='0 0 0' update_rate:=100.0">
     <!-- Create a pressure plate link -->
     <link name="${sensor_name}_link">
@@ -34,5 +34,5 @@
         <origin xyz="0 0 0" rpy="0 0 0"/>
         <geometry>
-          <box size="${box_size}"/>
+          <cylinder radius="0.007" length="0.005"/>
         </geometry>
         <surface>
@@ -49,5 +49,5 @@
         <origin xyz="0 0 0" rpy="0 0 0"/>
         <geometry>
-          <box size="${box_size}"/>
+          <cylinder radius="0.007" length="0.005"/>
         </geometry>
         <material name="pressure_sensor_material">
@@ -64,12 +64,12 @@
       <child link="${sensor_name}_link"/>
       <origin xyz="${position}" rpy="${rpy}"/>
-      <axis xyz="0 0 1"/>  <!-- Can compress vertically only -->
-      <limit effort="10000.0" lower="-0.0001" upper="0.0001" velocity="0.01"/>
-      <dynamics damping="100000.0" friction="0.0"/>  <!-- Very stiff -->
+      <axis xyz="0 1 0"/>  <!-- Can compress vertically only -->
+      <limit effort="1000.0" lower="-0.001" upper="0.001" velocity="0.1"/>
+      <dynamics damping="100.0" friction="10.0"/>  <!-- Very stiff -->
     </joint>
     <!-- Gazebo: Make joint very stiff (like a load cell) -->
     <gazebo reference="${sensor_name}_joint">
       <implicitSpringDamper>true</implicitSpringDamper>
-      <springStiffness>1000000.0</springStiffness>  <!-- Very high stiffness -->
+      <springStiffness>100000.0</springStiffness>  <!-- Very high stiffness -->
       <springReference>0.0</springReference>
     </gazebo>
@@ -142,5 +142,5 @@
     - sensor_rpy: Roll Pitch Yaw orientation to align sensor flat on ground
   -->
-  <xacro:macro name="foot_contact_sensor" params="foot_link prefix foot_bottom_offset:='-0.05' sensor_rpy:='0 0 0'">
+  <xacro:macro name="foot_contact_sensor" params="foot_link prefix position:='0 0 0' sensor_rpy:='0 0 0'">
     <!-- Force-torque sensor at bottom of foot (like a pressure plate) -->
     <xacro:force_torque_sensor
@@ -148,7 +148,6 @@
       sensor_name="${prefix}_foot_contact"
       topic="/${prefix}_foot/contact"
-      position="0 ${foot_bottom_offset} 0"
+      position="${position}"
       rpy="${sensor_rpy}"
-      box_size="0.08 0.06 0.01"
       update_rate="100.0"/>
   </xacro:macro>
