Commit message: updated robot.urdf with the new paths

File: src/robot_description/humanoid_description/urdf/robot.urdf (robot description, URDF)
Before this commit: robot assy_forurdf_kdheadless, 23 links, 22 joints
Links:
- link KC_C_101R_ShldYokeDrive: geometry collision mesh filename=meshes/collision/KC_C_101R_ShldYokeDrive.collision.stl; visual mesh filename=meshes/visual/KC_C_101R_ShldYokeDrive.stl
- link KC_C_202R: geometry collision mesh filename=meshes/collision/KC_C_202R.collision.stl; visual mesh filename=meshes/visual/KC_C_202R.stl
- link KC_C_401L_Up_Forearm_Drive: geometry collision mesh filename=meshes/collision/KC_C_401L_Up_Forearm_Drive.collision.stl; visual mesh filename=meshes/visual/KC_C_401L_Up_Forearm_Drive.stl
- link KC_C_401R_R_UpForearmDrive: geometry collision mesh filename=meshes/collision/KC_C_401R_R_UpForearmDrive.collision.stl; visual mesh filename=meshes/visual/KC_C_401R_R_UpForearmDrive.stl
- link KD_B_102B_TORSO_BTM: geometry collision mesh filename=meshes/collision/KD_B_102B_TORSO_BTM.collision.stl; visual mesh filename=meshes/visual/KD_B_102B_TORSO_BTM.stl
- link KD_C_101L_ShldYokeDrive: geometry collision mesh filename=meshes/collision/KD_C_101L_ShldYokeDrive.collision.stl; visual mesh filename=meshes/visual/KD_C_101L_ShldYokeDrive.stl
- link KD_C_301L_LowerBicepDrive: geometry collision mesh filename=meshes/collision/KD_C_301L_LowerBicepDrive.collision.stl; visual mesh filename=meshes/visual/KD_C_301L_LowerBicepDrive.stl
- link KD_D_102L_L_Hip_Yoke_Drive: geometry collision mesh filename=meshes/collision/KD_D_102L_L_Hip_Yoke_Drive.collision.stl; visual mesh filename=meshes/visual/KD_D_102L_L_Hip_Yoke_Drive.stl
- link KD_D_102R: geometry collision mesh filename=meshes/collision/KD_D_102R.collision.stl; visual mesh filename=meshes/visual/KD_D_102R.stl
- link KD_D_301L_L_Femur_Lower_Drive: geometry collision mesh filename=meshes/collision/KD_D_301L_L_Femur_Lower_Drive.collision.stl; visual mesh filename=meshes/visual/KD_D_301L_L_Femur_Lower_Drive.stl
- link KD_D_301R: geometry collision mesh filename=meshes/collision/KD_D_301R.collision.stl; visual mesh filename=meshes/visual/KD_D_301R.stl
- link KD_D_401L_L_Shin_Drive: geometry collision mesh filename=meshes/collision/KD_D_401L_L_Shin_Drive.collision.stl; visual mesh filename=meshes/visual/KD_D_401L_L_Shin_Drive.stl
- link KD_D_401R: geometry collision mesh filename=meshes/collision/KD_D_401R.collision.stl; visual mesh filename=meshes/visual/KD_D_401R.stl
- link LFootBushing_GPF_1517_12: geometry collision mesh filename=meshes/collision/LFootBushing_GPF_1517_12.collision.stl; visual mesh filename=meshes/visual/LFootBushing_GPF_1517_12.stl
- link L_Hip_Roll_RS03: geometry collision mesh filename=meshes/collision/L_Hip_Roll_RS03.collision.stl; visual mesh filename=meshes/visual/L_Hip_Roll_RS03.stl
- link L_Hip_Roll_RS03_2: geometry collision mesh filename=meshes/collision/L_Hip_Roll_RS03_2.collision.stl; visual mesh filename=meshes/visual/L_Hip_Roll_RS03_2.stl
- link PRT0001: geometry collision mesh filename=meshes/collision/PRT0001.collision.stl; visual mesh filename=meshes/visual/PRT0001.stl
- link PRT0001_2: geometry collision mesh filename=meshes/collision/PRT0001_2.collision.stl; visual mesh filename=meshes/visual/PRT0001_2.stl
- link RFootBushing_GPF_1517_12: geometry collision mesh filename=meshes/collision/RFootBushing_GPF_1517_12.collision.stl; visual mesh filename=meshes/visual/RFootBushing_GPF_1517_12.stl
- link RS03_3: geometry collision mesh filename=meshes/collision/RS03_3.collision.stl; visual mesh filename=meshes/visual/RS03_3.stl
- link RS03_4: geometry collision mesh filename=meshes/collision/RS03_4.collision.stl; visual mesh filename=meshes/visual/RS03_4.stl
- link imu: geometry collision mesh filename=meshes/collision/imu.collision.stl; visual mesh filename=meshes/visual/imu.stl

Commit message: fiex urdf mesh paths

File: src/robot_description/humanoid_description/urdf/robot.urdf (robot description, URDF)
Before this commit: robot assy_forurdf_kdheadless, 23 links, 22 joints
Links:
- link KC_C_101R_ShldYokeDrive: geometry collision mesh filename=package://humanoid_description/meshes/collision/KC_C_101R_S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; visual mesh filename=package://humanoid_description/meshes/visual/KC_C_101R_Shld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
- link KC_C_202R: geometry collision mesh filename=package://humanoid_description/meshes/collision/KC_C_202R.c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; visual mesh filename=package://humanoid_description/meshes/visual/KC_C_202R.stl
- link KC_C_401L_Up_Forearm_Drive: geometry collision mesh filename=package://humanoid_description/meshes/collision/KC_C_401L_U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; visual mesh filename=package://humanoid_description/meshes/visual/KC_C_401L_Up_F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
- link KC_C_401R_R_UpForearmDrive: geometry collision mesh filename=package://humanoid_description/meshes/collision/KC_C_401R_R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; visual mesh filename=package://humanoid_description/meshes/visual/KC_C_401R_R_Up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
- link KD_B_102B_TORSO_BTM: geometry collision mesh filename=package://humanoid_description/meshes/collision/KD_B_102B_T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; visual mesh filename=package://humanoid_description/meshes/visual/KD_B_102B_TORS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
- link KD_C_101L_ShldYokeDrive: geometry collision mesh filename=package://humanoid_description/meshes/collision/KD_C_101L_S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; visual mesh filename=package://humanoid_description/meshes/visual/KD_C_101L_Shld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
- link KD_C_301L_LowerBicepDrive: geometry collision mesh filename=package://humanoid_description/meshes/collision/KD_C_301L_L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; visual mesh filename=package://humanoid_description/meshes/visual/KD_C_301L_Lowe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
- link KD_D_102L_L_Hip_Yoke_Drive: geometry collision mesh filename=package://humanoid_description/meshes/collision/KD_D_102L_L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; visual mesh filename=package://humanoid_description/meshes/visual/KD_D_102L_L_Hi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
- link KD_D_102R: geometry collision mesh filename=package://humanoid_description/meshes/collision/KD_D_102R.c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; visual mesh filename=package://humanoid_description/meshes/visual/KD_D_102R.stl
- link KD_D_301L_L_Femur_Lower_Drive: geometry collision mesh filename=package://humanoid_description/meshes/collision/KD_D_301L_L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; visual mesh filename=package://humanoid_description/meshes/visual/KD_D_301L_L_Fe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
- link KD_D_301R: geometry collision mesh filename=package://humanoid_description/meshes/collision/KD_D_301R.c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; visual mesh filename=package://humanoid_description/meshes/visual/KD_D_301R.stl
- link KD_D_401L_L_Shin_Drive: geometry collision mesh filename=package://humanoid_description/meshes/collision/KD_D_401L_L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; visual mesh filename=package://humanoid_description/meshes/visual/KD_D_401L_L_Sh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
- link KD_D_401R: geometry collision mesh filename=package://humanoid_description/meshes/collision/KD_D_401R.c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; visual mesh filename=package://humanoid_description/meshes/visual/KD_D_401R.stl
- link LFootBushing_GPF_1517_12: geometry collision mesh filename=package://humanoid_description/meshes/collision/LFootBushin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; visual mesh filename=package://humanoid_description/meshes/visual/LFootBushing_G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
- link L_Hip_Roll_RS03: geometry collision mesh filename=package://humanoid_description/meshes/collision/L_Hip_Roll_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; visual mesh filename=package://humanoid_description/meshes/visual/L_Hip_Roll_RS0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
- link L_Hip_Roll_RS03_2: geometry collision mesh filename=package://humanoid_description/meshes/collision/L_Hip_Roll_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; visual mesh filename=package://humanoid_description/meshes/visual/L_Hip_Roll_RS0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
- link PRT0001: geometry collision mesh filename=package://humanoid_description/meshes/collision/PRT0001.col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; visual mesh filename=package://humanoid_description/meshes/visual/PRT0001.stl
- link PRT0001_2: geometry collision mesh filename=package://humanoid_description/meshes/collision/PRT0001_2.c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; visual mesh filename=package://humanoid_description/meshes/visual/PRT0001_2.stl
- link RFootBushing_GPF_1517_12: geometry collision mesh filename=package://humanoid_description/meshes/collision/RFootBushin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; visual mesh filename=package://humanoid_description/meshes/visual/RFootBushing_G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
- link RS03_3: geometry collision mesh filename=package://humanoid_description/meshes/collision/RS03_3.coll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; visual mesh filename=package://humanoid_description/meshes/visual/RS03_3.stl
- link RS03_4: geometry collision mesh filename=package://humanoid_description/meshes/collision/RS03_4.coll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; visual mesh filename=package://humanoid_description/meshes/visual/RS03_4.stl
- link imu: geometry collision mesh filename=package://humanoid_description/meshes/collision/imu.collisi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; visual mesh filename=package://humanoid_description/meshes/visual/imu.stl

Commit message: g1 description

File: src/robot_description/humanoid_description/urdf/robot.urdf (robot description, URDF)
Before this commit: robot assy_forurdf_kdheadless, 23 links, 22 joints
Links:
- removed link KC_C_101R_ShldYokeDrive
- removed link KC_C_202R
- removed link KC_C_401L_Up_Forearm_Drive
- removed link KC_C_401R_R_UpForearmDrive
- removed link KD_B_102B_TORSO_BTM
- removed link KD_C_101L_ShldYokeDrive
- removed link KD_C_301L_LowerBicepDrive
- removed link KD_D_102L_L_Hip_Yoke_Drive
- removed link KD_D_102R
- removed link KD_D_301L_L_Femur_Lower_Drive
- removed link KD_D_301R
- removed link KD_D_401L_L_Shin_Drive
- removed link KD_D_401R
- removed link LFootBushing_GPF_1517_12
- removed link L_Hip_Roll_RS03
- removed link L_Hip_Roll_RS03_2
- removed link PRT0001
- removed link PRT0001_2
- removed link RFootBushing_GPF_1517_12
- removed link RS03_3
- removed link RS03_4
- removed link base
- removed link imu
- added link d435_link
- added link head_link, mass 1.036; collision mesh filename=meshes/head_link.STL; visual mesh filename=meshes/head_link.STL
- added link imu_in_pelvis
- added link imu_in_torso
- added link left_ankle_pitch_link, mass 0.074; collision mesh filename=meshes/left_ankle_pitch_link.STL; visual mesh filename=meshes/left_ankle_pitch_link.STL
- added link left_ankle_roll_link, mass 0.608; collision sphere radius=0.005; collision sphere radius=0.005
- added link left_elbow_link, mass 0.6; collision mesh filename=meshes/left_elbow_link.STL; visual mesh filename=meshes/left_elbow_link.STL
- added link left_hip_pitch_link, mass 1.35; collision mesh filename=meshes/left_hip_pitch_link.STL; visual mesh filename=meshes/left_hip_pitch_link.STL
- added link left_hip_roll_link, mass 1.52; collision mesh filename=meshes/left_hip_roll_link.STL; visual mesh filename=meshes/left_hip_roll_link.STL
- added link left_hip_yaw_link, mass 1.702; collision mesh filename=meshes/left_hip_yaw_link.STL; visual mesh filename=meshes/left_hip_yaw_link.STL
- added link left_knee_link, mass 1.932; collision mesh filename=meshes/left_knee_link.STL; visual mesh filename=meshes/left_knee_link.STL
- added link left_rubber_hand, mass 0.170; visual mesh filename=meshes/left_rubber_hand.STL
- added link left_shoulder_pitch_link, mass 0.718; collision cylinder length=0.05 radius=0.03; visual mesh filename=meshes/left_shoulder_pitch_link.STL
- added link left_shoulder_roll_link, mass 0.643; collision cylinder length=0.03 radius=0.03; visual mesh filename=meshes/left_shoulder_roll_link.STL
- added link left_shoulder_yaw_link, mass 0.734; collision mesh filename=meshes/left_shoulder_yaw_link.STL; visual mesh filename=meshes/left_shoulder_yaw_link.STL
- added link left_wrist_pitch_link, mass 0.48404956; collision mesh filename=meshes/left_wrist_pitch_link.STL; visual mesh filename=meshes/left_wrist_pitch_link.STL
- added link left_wrist_roll_link, mass 0.08544498; collision mesh filename=meshes/left_wrist_roll_link.STL; visual mesh filename=meshes/left_wrist_roll_link.STL
- added link left_wrist_yaw_link, mass 0.08457647; collision mesh filename=meshes/left_wrist_yaw_link.STL; visual mesh filename=meshes/left_wrist_yaw_link.STL
- added link logo_link, mass 0.001; collision mesh filename=meshes/logo_link.STL; visual mesh filename=meshes/logo_link.STL
- added link mid360_link
- added link pelvis, mass 3.813; visual mesh filename=meshes/pelvis.STL
- added link pelvis_contour_link, mass 0.001; collision mesh filename=meshes/pelvis_contour_link.STL; visual mesh filename=meshes/pelvis_contour_link.STL
- added link right_ankle_pitch_link, mass 0.074; collision mesh filename=meshes/right_ankle_pitch_link.STL; visual mesh filename=meshes/right_ankle_pitch_link.STL
- added link right_ankle_roll_link, mass 0.608; collision sphere radius=0.005; collision sphere radius=0.005
- added link right_elbow_link, mass 0.6; collision mesh filename=meshes/right_elbow_link.STL; visual mesh filename=meshes/right_elbow_link.STL
- added link right_hip_pitch_link, mass 1.35; collision mesh filename=meshes/right_hip_pitch_link.STL; visual mesh filename=meshes/right_hip_pitch_link.STL
- added link right_hip_roll_link, mass 1.52; collision mesh filename=meshes/right_hip_roll_link.STL; visual mesh filename=meshes/right_hip_roll_link.STL
- added link right_hip_yaw_link, mass 1.702; collision mesh filename=meshes/right_hip_yaw_link.STL; visual mesh filename=meshes/right_hip_yaw_link.STL
- added link right_knee_link, mass 1.932; collision mesh filename=meshes/right_knee_link.STL; visual mesh filename=meshes/right_knee_link.STL
- added link right_rubber_hand, mass 0.170; visual mesh filename=meshes/right_rubber_hand.STL
- added link right_shoulder_pitch_link, mass 0.718; collision cylinder length=0.05 radius=0.03; visual mesh filename=meshes/right_shoulder_pitch_link.STL
- added link right_shoulder_roll_link, mass 0.643; collision cylinder length=0.03 radius=0.03; visual mesh filename=meshes/right_shoulder_roll_link.STL
- added link right_shoulder_yaw_link, mass 0.734; collision mesh filename=meshes/right_shoulder_yaw_link.STL; visual mesh filename=meshes/right_shoulder_yaw_link.STL
- added link right_wrist_pitch_link, mass 0.48404956; collision mesh filename=meshes/right_wrist_pitch_link.STL; visual mesh filename=meshes/right_wrist_pitch_link.STL
- added link right_wrist_roll_link, mass 0.08544498; collision mesh filename=meshes/right_wrist_roll_link.STL; visual mesh filename=meshes/right_wrist_roll_link.STL
- added link right_wrist_yaw_link, mass 0.08457647; collision mesh filename=meshes/right_wrist_yaw_link.STL; visual mesh filename=meshes/right_wrist_yaw_link.STL
- added link torso_link, mass 8.562; collision mesh filename=meshes/torso_link.STL; visual mesh filename=meshes/torso_link.STL
- added link waist_roll_link, mass 0.047; visual mesh filename=meshes/waist_roll_link.STL
- added link waist_support_link, mass 0.001; collision mesh filename=meshes/waist_support_link.STL; visual mesh filename=meshes/waist_support_link.STL
- added link waist_yaw_link, mass 0.244; visual mesh filename=meshes/waist_yaw_link.STL
Joints:
- removed joint base_joint
- removed joint dof_left_ankle_02
- removed joint dof_left_elbow_02
- removed joint dof_left_hip_pitch_04
- removed joint dof_left_hip_roll_03
- removed joint dof_left_hip_yaw_03
- removed joint dof_left_knee_04
- removed joint dof_left_shoulder_pitch_03
- removed joint dof_left_shoulder_roll_03
- removed joint dof_left_shoulder_yaw_02
- removed joint dof_left_wrist_00
- removed joint dof_right_ankle_02
- removed joint dof_right_elbow_02
- removed joint dof_right_hip_pitch_04
- removed joint dof_right_hip_roll_03
- removed joint dof_right_hip_yaw_03
- removed joint dof_right_knee_04
- removed joint dof_right_shoulder_pitch_03
- removed joint dof_right_shoulder_roll_03
- removed joint dof_right_shoulder_yaw_02
- removed joint dof_right_wrist_00
- removed joint frame_imu_site
- added joint d435_joint: type fixed, parent torso_link, child d435_link, origin xyz=0.0576235 0.01753 0.41987 rpy=0 0.8307767239493009 0
- added joint head_joint: type fixed, parent torso_link, child head_link, origin xyz=0.0039635 0 -0.054 rpy=0 0 0
- added joint imu_in_pelvis_joint: type fixed, parent pelvis, child imu_in_pelvis, origin xyz=0.04525 0 -0.08339 rpy=0 0 0
- added joint imu_in_torso_joint: type fixed, parent torso_link, child imu_in_torso, origin xyz=-0.03959 -0.00224 0.13792 rpy=0 0 0
- added joint left_ankle_pitch_joint: type revolute, parent left_knee_link, child left_ankle_pitch_link, origin xyz=0 -9.4445E-05 -0.30001 rpy=0 0 0, axis 0 1 0, limit lower=-0.87267 upper=0.5236 effort=35 velocity=30
- added joint left_ankle_roll_joint: type revolute, parent left_ankle_pitch_link, child left_ankle_roll_link, origin xyz=0 0 -0.017558 rpy=0 0 0, axis 1 0 0, limit lower=-0.2618 upper=0.2618 effort=35 velocity=30
- added joint left_elbow_joint: type revolute, parent left_shoulder_yaw_link, child left_elbow_link, origin xyz=0.015783 0 -0.080518 rpy=0 0 0, axis 0 1 0, limit lower=-1.0472 upper=2.0944 effort=25 velocity=37
- added joint left_hand_palm_joint: type fixed, parent left_wrist_yaw_link, child left_rubber_hand, origin xyz=0.0415 0.003 0 rpy=0 0 0
- added joint left_hip_pitch_joint: type revolute, parent pelvis, child left_hip_pitch_link, origin xyz=0 0.064452 -0.1027 rpy=0 0 0, axis 0 1 0, limit lower=-2.5307 upper=2.8798 effort=88 velocity=32
- added joint left_hip_roll_joint: type revolute, parent left_hip_pitch_link, child left_hip_roll_link, origin xyz=0 0.052 -0.030465 rpy=0 -0.1749 0, axis 1 0 0, limit lower=-0.5236 upper=2.9671 effort=88 velocity=32
- added joint left_hip_yaw_joint: type revolute, parent left_hip_roll_link, child left_hip_yaw_link, origin xyz=0.025001 0 -0.12412 rpy=0 0 0, axis 0 0 1, limit lower=-2.7576 upper=2.7576 effort=88 velocity=32
- added joint left_knee_joint: type revolute, parent left_hip_yaw_link, child left_knee_link, origin xyz=-0.078273 0.0021489 -0.17734 rpy=0 0.1749 0, axis 0 1 0, limit lower=-0.087267 upper=2.8798 effort=139 velocity=20
- added joint left_shoulder_pitch_joint: type revolute, parent torso_link, child left_shoulder_pitch_link, origin xyz=0.0039563 0.10022 0.23778 rpy=0.27931 5.4949E-05 -0.00019159, axis 0 1 0, limit lower=-3.0892 upper=2.6704 effort=25 velocity=37
- added joint left_shoulder_roll_joint: type revolute, parent left_shoulder_pitch_link, child left_shoulder_roll_link, origin xyz=0 0.038 -0.013831 rpy=-0.27925 0 0, axis 1 0 0, limit lower=-1.5882 upper=2.2515 effort=25 velocity=37
- added joint left_shoulder_yaw_joint: type revolute, parent left_shoulder_roll_link, child left_shoulder_yaw_link, origin xyz=0 0.00624 -0.1032 rpy=0 0 0, axis 0 0 1, limit lower=-2.618 upper=2.618 effort=25 velocity=37
- added joint left_wrist_pitch_joint: type revolute, parent left_wrist_roll_link, child left_wrist_pitch_link, origin xyz=0.038 0 0 rpy=0 0 0, axis 0 1 0, limit lower=-1.614429558 upper=1.614429558 effort=5 velocity=22
- added joint left_wrist_roll_joint: type revolute, parent left_elbow_link, child left_wrist_roll_link, origin xyz=0.100 0.00188791 -0.010 rpy=0 0 0, axis 1 0 0, limit lower=-1.972222054 upper=1.972222054 effort=25 velocity=37
- added joint left_wrist_yaw_joint: type revolute, parent left_wrist_pitch_link, child left_wrist_yaw_link, origin xyz=0.046 0 0 rpy=0 0 0, axis 0 0 1, limit lower=-1.614429558 upper=1.614429558 effort=5 velocity=22
- added joint logo_joint: type fixed, parent torso_link, child logo_link, origin xyz=0.0039635 0 -0.054 rpy=0 0 0
- added joint mid360_joint: type fixed, parent torso_link, child mid360_link, origin xyz=0.0002835 0.00003 0.40618 rpy=0 0.04014257279586953 0
- added joint pelvis_contour_joint: type fixed, parent pelvis, child pelvis_contour_link
- added joint right_ankle_pitch_joint: type revolute, parent right_knee_link, child right_ankle_pitch_link, origin xyz=0 9.4445E-05 -0.30001 rpy=0 0 0, axis 0 1 0, limit lower=-0.87267 upper=0.5236 effort=35 velocity=30
- added joint right_ankle_roll_joint: type revolute, parent right_ankle_pitch_link, child right_ankle_roll_link, origin xyz=0 0 -0.017558 rpy=0 0 0, axis 1 0 0, limit lower=-0.2618 upper=0.2618 effort=35 velocity=30
- added joint right_elbow_joint: type revolute, parent right_shoulder_yaw_link, child right_elbow_link, origin xyz=0.015783 0 -0.080518 rpy=0 0 0, axis 0 1 0, limit lower=-1.0472 upper=2.0944 effort=25 velocity=37
- added joint right_hand_palm_joint: type fixed, parent right_wrist_yaw_link, child right_rubber_hand, origin xyz=0.0415 -0.003 0 rpy=0 0 0
- added joint right_hip_pitch_joint: type revolute, parent pelvis, child right_hip_pitch_link, origin xyz=0 -0.064452 -0.1027 rpy=0 0 0, axis 0 1 0, limit lower=-2.5307 upper=2.8798 effort=88 velocity=32
- added joint right_hip_roll_joint: type revolute, parent right_hip_pitch_link, child right_hip_roll_link, origin xyz=0 -0.052 -0.030465 rpy=0 -0.1749 0, axis 1 0 0, limit lower=-2.9671 upper=0.5236 effort=88 velocity=32
- added joint right_hip_yaw_joint: type revolute, parent right_hip_roll_link, child right_hip_yaw_link, origin xyz=0.025001 0 -0.12412 rpy=0 0 0, axis 0 0 1, limit lower=-2.7576 upper=2.7576 effort=88 velocity=32
- added joint right_knee_joint: type revolute, parent right_hip_yaw_link, child right_knee_link, origin xyz=-0.078273 -0.0021489 -0.17734 rpy=0 0.1749 0, axis 0 1 0, limit lower=-0.087267 upper=2.8798 effort=139 velocity=20
- added joint right_shoulder_pitch_joint: type revolute, parent torso_link, child right_shoulder_pitch_link, origin xyz=0.0039563 -0.10021 0.23778 rpy=-0.27931 5.4949E-05 0.00019159, axis 0 1 0, limit lower=-3.0892 upper=2.6704 effort=25 velocity=37
- added joint right_shoulder_roll_joint: type revolute, parent right_shoulder_pitch_link, child right_shoulder_roll_link, origin xyz=0 -0.038 -0.013831 rpy=0.27925 0 0, axis 1 0 0, limit lower=-2.2515 upper=1.5882 effort=25 velocity=37
- added joint right_shoulder_yaw_joint: type revolute, parent right_shoulder_roll_link, child right_shoulder_yaw_link, origin xyz=0 -0.00624 -0.1032 rpy=0 0 0, axis 0 0 1, limit lower=-2.618 upper=2.618 effort=25 velocity=37
- added joint right_wrist_pitch_joint: type revolute, parent right_wrist_roll_link, child right_wrist_pitch_link, origin xyz=0.038 0 0 rpy=0 0 0, axis 0 1 0, limit lower=-1.614429558 upper=1.614429558 effort=5 velocity=22
- added joint right_wrist_roll_joint: type revolute, parent right_elbow_link, child right_wrist_roll_link, origin xyz=0.100 -0.00188791 -0.010 rpy=0 0 0, axis 1 0 0, limit lower=-1.972222054 upper=1.972222054 effort=25 velocity=37
- added joint right_wrist_yaw_joint: type revolute, parent right_wrist_pitch_link, child right_wrist_yaw_link, origin xyz=0.046 0 0 rpy=0 0 0, axis 0 0 1, limit lower=-1.614429558 upper=1.614429558 effort=5 velocity=22
- added joint waist_pitch_joint: type fixed, parent waist_roll_link, child torso_link, origin xyz=0 0 0.019 rpy=0 0 0, axis 0 1 0, limit lower=-0.52 upper=0.52 effort=35 velocity=30
- added joint waist_roll_joint: type fixed, parent waist_yaw_link, child waist_roll_link, origin xyz=-0.0039635 0 0.035 rpy=0 0 0, axis 1 0 0, limit lower=-0.52 upper=0.52 effort=35 velocity=30
- added joint waist_support_joint: type fixed, parent torso_link, child waist_support_link, origin xyz=0.0039635 0 -0.054 rpy=0 0 0
- added joint waist_yaw_joint: type revolute, parent pelvis, child waist_yaw_link, origin xyz=0 0 0 rpy=0 0 0, axis 0 0 1, limit lower=-2.618 upper=2.618 effort=88 velocity=32
