Commit message: Add torso_ref frame for stable torso orientation task

File: src/robot_description/humanoid_description/urdf/robot_mc_rtc.urdf (robot description, URDF)
Before this commit: robot g1_29dof_lock_waist, 40 links, 39 joints
Links:
- added link torso_ref
Joints:
- added joint torso_ref_joint: type fixed, parent torso_link, child torso_ref, origin xyz=0.00331658 0.000261533 0.179856 rpy=0 0 0
