Commit message: link mesh path corection

File: src/robot_description/humanoid_description/xacro/links/robot_links.xacro (robot description, xacro)
@@ -10,5 +10,5 @@
             <origin xyz="0 0 0" rpy="0 0 0" />
             <geometry>
-                <mesh filename="package://humanoid_description/urdf/package://humanoid_description/urdf/meshes/pelvis.STL" />
+                <mesh filename="package://humanoid_description/meshes/pelvis.STL" />
             </geometry>
             <material name="dark" />
@@ -24,12 +24,12 @@
             <origin xyz="0 0 0" rpy="0 0 0" />
             <geometry>
-                <mesh filename="package://humanoid_description/urdf/meshes/pelvis_contour_link.STL" />
-            </geometry>
-            <material name="white" />
-        </visual>
-        <collision>
-            <origin xyz="0 0 0" rpy="0 0 0" />
-            <geometry>
-                <mesh filename="package://humanoid_description/urdf/meshes/pelvis_contour_link.STL" />
+                <mesh filename="package://humanoid_description/meshes/pelvis_contour_link.STL" />
+            </geometry>
+            <material name="white" />
+        </visual>
+        <collision>
+            <origin xyz="0 0 0" rpy="0 0 0" />
+            <geometry>
+                <mesh filename="package://humanoid_description/meshes/pelvis_contour_link.STL" />
             </geometry>
         </collision>
@@ -44,5 +44,5 @@
             <origin xyz="0 0 0" rpy="0 0 0" />
             <geometry>
-                <mesh filename="package://humanoid_description/urdf/meshes/left_hip_pitch_link.STL" />
+                <mesh filename="package://humanoid_description/meshes/left_hip_pitch_link.STL" />
             </geometry>
             <material name="dark" />
@@ -51,5 +51,5 @@
             <origin xyz="0 0 0" rpy="0 0 0" />
             <geometry>
-                <mesh filename="package://humanoid_description/urdf/meshes/left_hip_pitch_link.STL" />
+                <mesh filename="package://humanoid_description/meshes/left_hip_pitch_link.STL" />
             </geometry>
         </collision>
@@ -64,12 +64,12 @@
             <origin xyz="0 0 0" rpy="0 0 0" />
             <geometry>
-                <mesh filename="package://humanoid_description/urdf/meshes/left_hip_roll_link.STL" />
-            </geometry>
-            <material name="white" />
-        </visual>
-        <collision>
-            <origin xyz="0 0 0" rpy="0 0 0" />
-            <geometry>
-                <mesh filename="package://humanoid_description/urdf/meshes/left_hip_roll_link.STL" />
+                <mesh filename="package://humanoid_description/meshes/left_hip_roll_link.STL" />
+            </geometry>
+            <material name="white" />
+        </visual>
+        <collision>
+            <origin xyz="0 0 0" rpy="0 0 0" />
+            <geometry>
+                <mesh filename="package://humanoid_description/meshes/left_hip_roll_link.STL" />
             </geometry>
         </collision>
@@ -84,12 +84,12 @@
             <origin xyz="0 0 0" rpy="0 0 0" />
             <geometry>
-                <mesh filename="package://humanoid_description/urdf/meshes/left_hip_yaw_link.STL" />
-            </geometry>
-            <material name="white" />
-        </visual>
-        <collision>
-            <origin xyz="0 0 0" rpy="0 0 0" />
-            <geometry>
-                <mesh filename="package://humanoid_description/urdf/meshes/left_hip_yaw_link.STL" />
+                <mesh filename="package://humanoid_description/meshes/left_hip_yaw_link.STL" />
+            </geometry>
+            <material name="white" />
+        </visual>
+        <collision>
+            <origin xyz="0 0 0" rpy="0 0 0" />
+            <geometry>
+                <mesh filename="package://humanoid_description/meshes/left_hip_yaw_link.STL" />
             </geometry>
         </collision>
@@ -104,12 +104,12 @@
             <origin xyz="0 0 0" rpy="0 0 0" />
             <geometry>
-                <mesh filename="package://humanoid_description/urdf/meshes/left_knee_link.STL" />
-            </geometry>
-            <material name="white" />
-        </visual>
-        <collision>
-            <origin xyz="0 0 0" rpy="0 0 0" />
-            <geometry>
-                <mesh filename="package://humanoid_description/urdf/meshes/left_knee_link.STL" />
+                <mesh filename="package://humanoid_description/meshes/left_knee_link.STL" />
+            </geometry>
+            <material name="white" />
+        </visual>
+        <collision>
+            <origin xyz="0 0 0" rpy="0 0 0" />
+            <geometry>
+                <mesh filename="package://humanoid_description/meshes/left_knee_link.STL" />
             </geometry>
         </collision>
@@ -124,12 +124,12 @@
             <origin xyz="0 0 0" rpy="0 0 0" />
             <geometry>
-                <mesh filename="package://humanoid_description/urdf/meshes/left_ankle_pitch_link.STL" />
-            </geometry>
-            <material name="white" />
-        </visual>
-        <collision>
-            <origin xyz="0 0 0" rpy="0 0 0" />
-            <geometry>
-                <mesh filename="package://humanoid_description/urdf/meshes/left_ankle_pitch_link.STL" />
+                <mesh filename="package://humanoid_description/meshes/left_ankle_pitch_link.STL" />
+            </geometry>
+            <material name="white" />
+        </visual>
+        <collision>
+            <origin xyz="0 0 0" rpy="0 0 0" />
+            <geometry>
+                <mesh filename="package://humanoid_description/meshes/left_ankle_pitch_link.STL" />
             </geometry>
         </collision>
@@ -144,5 +144,5 @@
             <origin xyz="0 0 0" rpy="0 0 0" />
             <geometry>
-                <mesh filename="package://humanoid_description/urdf/meshes/left_ankle_roll_link.STL" />
+                <mesh filename="package://humanoid_description/meshes/left_ankle_roll_link.STL" />
             </geometry>
             <material name="dark" />
@@ -182,5 +182,5 @@
             <origin xyz="0 0 0" rpy="0 0 0" />
             <geometry>
-                <mesh filename="package://humanoid_description/urdf/meshes/right_hip_pitch_link.STL" />
+                <mesh filename="package://humanoid_description/meshes/right_hip_pitch_link.STL" />
             </geometry>
             <material name="dark" />
@@ -189,5 +189,5 @@
             <origin xyz="0 0 0" rpy="0 0 0" />
             <geometry>
-                <mesh filename="package://humanoid_description/urdf/meshes/right_hip_pitch_link.STL" />
+                <mesh filename="package://humanoid_description/meshes/right_hip_pitch_link.STL" />
             </geometry>
         </collision>
@@ -202,12 +202,12 @@
             <origin xyz="0 0 0" rpy="0 0 0" />
             <geometry>
-                <mesh filename="package://humanoid_description/urdf/meshes/right_hip_roll_link.STL" />
-            </geometry>
-            <material name="white" />
-        </visual>
-        <collision>
-            <origin xyz="0 0 0" rpy="0 0 0" />
-            <geometry>
-                <mesh filename="package://humanoid_description/urdf/meshes/right_hip_roll_link.STL" />
+                <mesh filename="package://humanoid_description/meshes/right_hip_roll_link.STL" />
+            </geometry>
+            <material name="white" />
+        </visual>
+        <collision>
+            <origin xyz="0 0 0" rpy="0 0 0" />
+            <geometry>
+                <mesh filename="package://humanoid_description/meshes/right_hip_roll_link.STL" />
             </geometry>
         </collision>
@@ -222,12 +222,12 @@
             <origin xyz="0 0 0" rpy="0 0 0" />
             <geometry>
-                <mesh filename="package://humanoid_description/urdf/meshes/right_hip_yaw_link.STL" />
-            </geometry>
-            <material name="white" />
-        </visual>
-        <collision>
-            <origin xyz="0 0 0" rpy="0 0 0" />
-            <geometry>
-                <mesh filename="package://humanoid_description/urdf/meshes/right_hip_yaw_link.STL" />
+                <mesh filename="package://humanoid_description/meshes/right_hip_yaw_link.STL" />
+            </geometry>
+            <material name="white" />
+        </visual>
+        <collision>
+            <origin xyz="0 0 0" rpy="0 0 0" />
+            <geometry>
+                <mesh filename="package://humanoid_description/meshes/right_hip_yaw_link.STL" />
             </geometry>
         </collision>
@@ -242,12 +242,12 @@
             <origin xyz="0 0 0" rpy="0 0 0" />
             <geometry>
-                <mesh filename="package://humanoid_description/urdf/meshes/right_knee_link.STL" />
-            </geometry>
-            <material name="white" />
-        </visual>
-        <collision>
-            <origin xyz="0 0 0" rpy="0 0 0" />
-            <geometry>
-                <mesh filename="package://humanoid_description/urdf/meshes/right_knee_link.STL" />
+                <mesh filename="package://humanoid_description/meshes/right_knee_link.STL" />
+            </geometry>
+            <material name="white" />
+        </visual>
+        <collision>
+            <origin xyz="0 0 0" rpy="0 0 0" />
+            <geometry>
+                <mesh filename="package://humanoid_description/meshes/right_knee_link.STL" />
             </geometry>
         </collision>
@@ -262,12 +262,12 @@
             <origin xyz="0 0 0" rpy="0 0 0" />
             <geometry>
-                <mesh filename="package://humanoid_description/urdf/meshes/right_ankle_pitch_link.STL" />
-            </geometry>
-            <material name="white" />
-        </visual>
-        <collision>
-            <origin xyz="0 0 0" rpy="0 0 0" />
-            <geometry>
-                <mesh filename="package://humanoid_description/urdf/meshes/right_ankle_pitch_link.STL" />
+                <mesh filename="package://humanoid_description/meshes/right_ankle_pitch_link.STL" />
+            </geometry>
+            <material name="white" />
+        </visual>
+        <collision>
+            <origin xyz="0 0 0" rpy="0 0 0" />
+            <geometry>
+                <mesh filename="package://humanoid_description/meshes/right_ankle_pitch_link.STL" />
             </geometry>
         </collision>
@@ -282,5 +282,5 @@
             <origin xyz="0 0 0" rpy="0 0 0" />
             <geometry>
-                <mesh filename="package://humanoid_description/urdf/meshes/right_ankle_roll_link.STL" />
+                <mesh filename="package://humanoid_description/meshes/right_ankle_roll_link.STL" />
             </geometry>
             <material name="dark" />
@@ -320,5 +320,5 @@
             <origin xyz="0 0 0" rpy="0 0 0" />
             <geometry>
-                <mesh filename="package://humanoid_description/urdf/meshes/waist_yaw_link.STL" />
+                <mesh filename="package://humanoid_description/meshes/waist_yaw_link.STL" />
             </geometry>
             <material name="white" />
@@ -334,5 +334,5 @@
             <origin xyz="0 0 0" rpy="0 0 0" />
             <geometry>
-                <mesh filename="package://humanoid_description/urdf/meshes/waist_roll_link.STL" />
+                <mesh filename="package://humanoid_description/meshes/waist_roll_link.STL" />
             </geometry>
             <material name="white" />
@@ -348,12 +348,12 @@
             <origin xyz="0 0 0" rpy="0 0 0" />
             <geometry>
-                <mesh filename="package://humanoid_description/urdf/meshes/torso_link.STL" />
-            </geometry>
-            <material name="white" />
-        </visual>
-        <collision>
-            <origin xyz="0 0 0" rpy="0 0 0" />
-            <geometry>
-                <mesh filename="package://humanoid_description/urdf/meshes/torso_link.STL" />
+                <mesh filename="package://humanoid_description/meshes/torso_link.STL" />
+            </geometry>
+            <material name="white" />
+        </visual>
+        <collision>
+            <origin xyz="0 0 0" rpy="0 0 0" />
+            <geometry>
+                <mesh filename="package://humanoid_description/meshes/torso_link.STL" />
             </geometry>
         </collision>
@@ -368,5 +368,5 @@
             <origin xyz="0 0 0" rpy="0 0 0" />
             <geometry>
-                <mesh filename="package://humanoid_description/urdf/meshes/logo_link.STL" />
+                <mesh filename="package://humanoid_description/meshes/logo_link.STL" />
             </geometry>
             <material name="dark" />
@@ -375,5 +375,5 @@
             <origin xyz="0 0 0" rpy="0 0 0" />
             <geometry>
-                <mesh filename="package://humanoid_description/urdf/meshes/logo_link.STL" />
+                <mesh filename="package://humanoid_description/meshes/logo_link.STL" />
             </geometry>
         </collision>
@@ -388,5 +388,5 @@
             <origin xyz="0 0 0" rpy="0 0 0" />
             <geometry>
-                <mesh filename="package://humanoid_description/urdf/meshes/head_link.STL" />
+                <mesh filename="package://humanoid_description/meshes/head_link.STL" />
             </geometry>
             <material name="dark" />
@@ -395,5 +395,5 @@
             <origin xyz="0 0 0" rpy="0 0 0" />
             <geometry>
-                <mesh filename="package://humanoid_description/urdf/meshes/head_link.STL" />
+                <mesh filename="package://humanoid_description/meshes/head_link.STL" />
             </geometry>
         </collision>
@@ -408,12 +408,12 @@
             <origin xyz="0 0 0" rpy="0 0 0" />
             <geometry>
-                <mesh filename="package://humanoid_description/urdf/meshes/waist_support_link.STL" />
-            </geometry>
-            <material name="white" />
-        </visual>
-        <collision>
-            <origin xyz="0 0 0" rpy="0 0 0" />
-            <geometry>
-                <mesh filename="package://humanoid_description/urdf/meshes/waist_support_link.STL" />
+                <mesh filename="package://humanoid_description/meshes/waist_support_link.STL" />
+            </geometry>
+            <material name="white" />
+        </visual>
+        <collision>
+            <origin xyz="0 0 0" rpy="0 0 0" />
+            <geometry>
+                <mesh filename="package://humanoid_description/meshes/waist_support_link.STL" />
             </geometry>
         </collision>
@@ -432,5 +432,5 @@
             <origin xyz="0 0 0" rpy="0 0 0" />
             <geometry>
-                <mesh filename="package://humanoid_description/urdf/meshes/left_shoulder_pitch_link.STL" />
+                <mesh filename="package://humanoid_description/meshes/left_shoulder_pitch_link.STL" />
             </geometry>
             <material name="white" />
@@ -452,5 +452,5 @@
             <origin xyz="0 0 0" rpy="0 0 0" />
             <geometry>
-                <mesh filename="package://humanoid_description/urdf/meshes/left_shoulder_roll_link.STL" />
+                <mesh filename="package://humanoid_description/meshes/left_shoulder_roll_link.STL" />
             </geometry>
             <material name="white" />
@@ -472,12 +472,12 @@
             <origin xyz="0 0 0" rpy="0 0 0" />
             <geometry>
-                <mesh filename="package://humanoid_description/urdf/meshes/left_shoulder_yaw_link.STL" />
-            </geometry>
-            <material name="white" />
-        </visual>
-        <collision>
-            <origin xyz="0 0 0" rpy="0 0 0" />
-            <geometry>
-                <mesh filename="package://humanoid_description/urdf/meshes/left_shoulder_yaw_link.STL" />
+                <mesh filename="package://humanoid_description/meshes/left_shoulder_yaw_link.STL" />
+            </geometry>
+            <material name="white" />
+        </visual>
+        <collision>
+            <origin xyz="0 0 0" rpy="0 0 0" />
+            <geometry>
+                <mesh filename="package://humanoid_description/meshes/left_shoulder_yaw_link.STL" />
             </geometry>
         </collision>
@@ -492,12 +492,12 @@
             <origin xyz="0 0 0" rpy="0 0 0" />
             <geometry>
-                <mesh filename="package://humanoid_description/urdf/meshes/left_elbow_link.STL" />
-            </geometry>
-            <material name="white" />
-        </visual>
-        <collision>
-            <origin xyz="0 0 0" rpy="0 0 0" />
-            <geometry>
-                <mesh filename="package://humanoid_description/urdf/meshes/left_elbow_link.STL" />
+                <mesh filename="package://humanoid_description/meshes/left_elbow_link.STL" />
+            </geometry>
+            <material name="white" />
+        </visual>
+        <collision>
+            <origin xyz="0 0 0" rpy="0 0 0" />
+            <geometry>
+                <mesh filename="package://humanoid_description/meshes/left_elbow_link.STL" />
             </geometry>
         </collision>
@@ -512,12 +512,12 @@
             <origin xyz="0 0 0" rpy="0 0 0" />
             <geometry>
-                <mesh filename="package://humanoid_description/urdf/meshes/left_wrist_roll_link.STL" />
-            </geometry>
-            <material name="white" />
-        </visual>
-        <collision>
-            <origin xyz="0 0 0" rpy="0 0 0" />
-            <geometry>
-                <mesh filename="package://humanoid_description/urdf/meshes/left_wrist_roll_link.STL" />
+                <mesh filename="package://humanoid_description/meshes/left_wrist_roll_link.STL" />
+            </geometry>
+            <material name="white" />
+        </visual>
+        <collision>
+            <origin xyz="0 0 0" rpy="0 0 0" />
+            <geometry>
+                <mesh filename="package://humanoid_description/meshes/left_wrist_roll_link.STL" />
             </geometry>
         </collision>
@@ -532,12 +532,12 @@
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